File: hardware/pikocore_gamepad/pcb/pikocore_gamepad.kicad_pcb (KiCad board)
At the start: 4 copper layers, 100 x 80 mm, 72 parts, among them J1 PHONES, J4 LCD_FPC, J5 SPEAKER 8R, Q1 2N7002, SW1 DPAD_UP, SW10 BTN_R, SW11 BTN_START, SW12 BTN_SELECT, SW15 PWR, SW2 DPAD_DOWN, SW3 DPAD_LEFT, SW4 DPAD_RIGHT, SW5 BTN_X, SW6 BTN_Y, SW7 BTN_A, SW8 BTN_B, SW9 BTN_L, U1 RP2350-Plus-16MB, U2 TPS61023DRLR, U3 PT2308-S, U4 PAM8302A, U5 PCM5102APWR

Commit message: hw: RP2350A chip-down en la placa (reemplaza el modulo RP2350-Plus)
El modulo Waveshare RP2350-Plus sale y su circuito pasa al dorso:
RP2350A QFN-60 con el nucleo de la placa minima oficial de Raspberry Pi
(MIT) copiado como bloque rigido (import_rp_minimal.py -> rp_core_ref.py,
colocado por rp_core.py), flash W25Q128, cristal 12 MHz, USB-C, cargador
ETA6096, OR de alimentacion con MBR230, buck-boost TPS63001 a 3V3,
botones BOOTSEL/RUN y pads SWD. GP0-22/GP26 sin cambios; GP23/24/29
nuevos (BB_PS, VBUS_SENSE, VSYS_ADC) tambien en config.h.

Ruteo:
- El cobre previo (nucleo, pistas manuales, vias a plano) va al DSN
  protegido; las zonas del nucleo en la cara del chip van como keepout.
- Segunda pasada de freerouting solo si deja menos conexiones abiertas.
- Senales a 0.127/0.127 con via 0.45/0.2; Power con via propia 0.6/0.3.
- Carriles de salida de la placa oficial para LCD_DC, LCD_MOSI,
  BTN_START y DPAD_UP/DOWN; pin 1 de U1 al anillo de 3V3 a mano.
- TPS63001 a 180 grados con L1/L2 a mano; GND y VBUS del USB-C a mano.

Puertas: 191 tests, ERC 0, DRC 0 errores / 0 sin conectar / 0 paridad
(9 avisos previos), G-5/G-4/G-2/placement en verde. G-0 sigue en rojo
solo por LCD_FPC_PIN_ORDER, como en main. Sin verificar: LCSC de R31
(ISET 150k), saturacion de L4, rotaciones del CPL de las piezas nuevas.

Co-Authored-By: Claude Opus 5.5 <noreply@anthropic.com>
Parts:
- added C32: 4.7uF, rp_minimal:generic_capc1005x50_wide, B.Cu at (23.4, 22.5)
- added C33: 4.7uF, rp_minimal:generic_capc1005x50_wide, B.Cu at (22.4, 22.5)
- added C34: 4.7uF, rp_minimal:generic_capc1005x50, B.Cu at (22.9, 24.7)
- added C35: 100nF, rp_minimal:generic_capc1005x50, B.Cu at (27.0, 14.0)
- added C36: 100nF, rp_minimal:generic_capc1005x50, B.Cu at (34.9, 21.3)
- added C37: 100nF, rp_minimal:generic_capc1005x50, B.Cu at (27.4, 27.6)
- added C38: 100nF, rp_minimal:generic_capc1005x50, B.Cu at (20.6, 18.4)
- added C39: 100nF, rp_minimal:generic_capc1005x50, B.Cu at (24.6, 14.0)
- added C40: 100nF, rp_minimal:generic_capc1005x50, B.Cu at (28.4, 27.6)
- added C41: 100nF, rp_minimal:generic_capc1005x50, B.Cu at (29.4, 14.0)
- added C42: 100nF, rp_minimal:generic_capc1005x50, B.Cu at (32.0, 26.2)
- added C43: 100nF, rp_minimal:generic_capc1005x50, B.Cu at (25.0, 27.0)
- added C44: 100nF, rp_minimal:generic_capc1005x50, B.Cu at (34.1, 18.7)
- added C45: 15pF, rp_minimal:generic_capc1005x50, B.Cu at (37.0, 19.1)
- added C46: 15pF, rp_minimal:generic_capc1005x50, B.Cu at (37.0, 22.1)
- added C47: 100nF, rp_minimal:generic_capc1005x50, B.Cu at (10.8, 16.7)
- added C48: 1uF, Capacitor_SMD:C_0603_1608Metric, B.Cu at (2.00, 30.0)
- added C49: 22uF, Capacitor_SMD:C_0805_2012Metric, B.Cu at (10.2, 30.5)
- added C50: 10uF, Capacitor_SMD:C_0603_1608Metric, B.Cu at (10.2, 35.6)
- added C51: 10uF, Capacitor_SMD:C_0603_1608Metric, B.Cu at (37.7, 36.9)
- added C52: 10uF, Capacitor_SMD:C_0603_1608Metric, B.Cu at (37.7, 30.4)
- added C53: 10uF, Capacitor_SMD:C_0603_1608Metric, B.Cu at (41.0, 30.4)
- added C54: 100nF, Capacitor_SMD:C_0603_1608Metric, B.Cu at (35.0, 29.8)
- added C55: 100nF, Capacitor_SMD:C_0603_1608Metric, B.Cu at (64.5, 42.8)
- added D1: MBR230LSFT1G, Diode_SMD:D_SOD-123F, B.Cu at (11.0, 26.5)
- added D2: MBR230LSFT1G, Diode_SMD:D_SOD-123F, B.Cu at (14.5, 35.6)
- added J2: USB-C, Connector_USB:USB_C_Receptacle_HCTL_HC-TYPE-C-16P-01A, B.Cu at (4.60, 19.4)
- added J3: LiPo, Connector_Molex:Molex_PicoBlade_53398-0271_1x02-1MP_P1.25mm_Vertical, B.Cu at (6.00, 45.0)
- added L3: 3.3uH, rp_minimal:abracon_aota-b201610s3r3-101-t, B.Cu at (20.8, 22.5)
- added L4: 2.2uH, Inductor_SMD:L_1210_3225Metric, B.Cu at (6.00, 35.6)
- added L5: 2.2uH, Inductor_SMD:L_1210_3225Metric, B.Cu at (40.2, 33.5)
- added R23: 33R, rp_minimal:generic_resc1005x35, B.Cu at (21.1, 24.7)
- added R24: 1k, rp_minimal:generic_resc1005x35, B.Cu at (34.9, 20.1)
- added R25: 27R, rp_minimal:generic_resc1005x35, B.Cu at (20.6, 19.4)
- added R26: 27R, rp_minimal:generic_resc1005x35, B.Cu at (20.6, 20.4)
- added R27: 1k, rp_minimal:generic_resc1005x35, B.Cu at (9.30, 9.40)
- added R28: 0R, rp_minimal:generic_resc1005x35, B.Cu at (10.7, 9.40)
- added R29: 5.1k, Resistor_SMD:R_0603_1608Metric, B.Cu at (3.00, 12.8)
- added R30: 5.1k, Resistor_SMD:R_0603_1608Metric, B.Cu at (3.00, 26.0)
- added R31: 150k, Resistor_SMD:R_0603_1608Metric, B.Cu at (2.00, 33.4)
- added R32: 100R, Resistor_SMD:R_0603_1608Metric, B.Cu at (32.8, 30.1)
- added R33: 100k, Resistor_SMD:R_0603_1608Metric, B.Cu at (32.8, 33.3)
- added R34: 10k, Resistor_SMD:R_0603_1608Metric, B.Cu at (32.8, 36.4)
- added R35: 100k, Resistor_SMD:R_0603_1608Metric, B.Cu at (60.5, 39.8)
- added R36: 200k, Resistor_SMD:R_0603_1608Metric, B.Cu at (64.5, 39.8)
- added R37: 200k, Resistor_SMD:R_0603_1608Metric, B.Cu at (56.5, 42.8)
- added R38: 100k, Resistor_SMD:R_0603_1608Metric, B.Cu at (60.5, 42.8)
- added SW13: BOOTSEL, Button_Switch_SMD:SW_Push_1P1T_XKB_TS-1187A, B.Cu at (5.50, 54.0)
- added SW14: RUN, Button_Switch_SMD:SW_Push_1P1T_XKB_TS-1187A, B.Cu at (5.50, 63.0)
- added TP1: SWCLK, TestPoint:TestPoint_Pad_D1.0mm, B.Cu at (59.0, 11.0)
- added TP2: SWDIO, TestPoint:TestPoint_Pad_D1.0mm, B.Cu at (86.0, 10.0)
- added TP3: GND, TestPoint:TestPoint_Pad_D1.0mm, B.Cu at (86.0, 13.0)
- added U6: W25Q128JVSIQ, rp_minimal:generic_soic127p790x195-8, B.Cu at (15.3, 13.6)
- added U7: TPS63001DRCR, Package_SON:Texas_DRC0010J_ThermalVias, B.Cu at (36.0, 33.5)
- added U8: ETA6096D3K, gamesetup_lcsc:DFN-10_L3.0-W3.0-P0.50-BL-EP2.4-1, B.Cu at (6.00, 31.0)
- added Y1: 12MHz, rp_minimal:generic_xtalcc320x250x80-4, B.Cu at (40.4, 20.5)
- U1: value RP2350-Plus-16MB -> RP2350A; footprint gamesetup_fp:RP2350-Plus_Socket -> rp_minimal:rpi_rp2350a_vias
- moved C23 68.0 mm to (74.8, 12.6)
- moved C24 57.9 mm to (74.8, 20.6)
- moved R14 57.5 mm to (34.5, 39.8)
- moved R17 55.2 mm to (38.5, 44.8)
- moved R16 54.1 mm to (34.5, 42.8)
- moved C26 51.6 mm to (33.5, 45.8)
- moved R13 47.8 mm to (41.5, 38.8)
- moved R15 43.9 mm to (38.5, 41.8)
- moved R18 43.9 mm to (42.5, 41.8)
- moved C12 41.2 mm to (82.5, 9.78)
- moved C25 41.0 mm to (42.5, 44.8)
- moved C27 33.2 mm to (56.5, 39.8)
- moved C8 32.6 mm to (54.5, 26.8)
- moved C9 31.8 mm to (58.5, 26.8)
- moved C18 29.4 mm to (83.5, 27.8)
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Connections:
- U1 pad 1: DPAD_UP -> 3V3
- U1 pad 11: I2S_DIN -> 3V3
- U1 pad 12: DPAD_RIGHT -> I2S_DIN
- U1 pad 13: GND -> DPAD_RIGHT
- U1 pad 18: GND -> BTN_START
- U1 pad 19: BTN_START -> BTN_SELECT
- U1 pad 2: DPAD_DOWN -> DPAD_UP
- U1 pad 20: BTN_SELECT -> 3V3
- U1 pad 21: I2S_BCK -> XIN
- U1 pad 22: I2S_LRCK -> XOUT
- U1 pad 23: GND -> 1V1
- U1 pad 24: BTN_L -> SWCLK
- U1 pad 25: BTN_R -> SWDIO
- U1 pad 26: SPK_SHDN -> RUN
- U1 pad 27: JACK_DET -> I2S_BCK
- U1 pad 28: GND -> I2S_LRCK
- U1 pad 29: DAC_XSMT -> BTN_L
- U1 pad 3: GND -> DPAD_DOWN
- U1 pad 30: unconnected-(U1-RUN-Pad30) -> 3V3
- U1 pad 31: LCD_TE -> BTN_R
- U1 pad 32: EXP_GP27 -> SPK_SHDN
- U1 pad 33: GND -> JACK_DET
- U1 pad 34: EXP_GP28 -> DAC_XSMT
- U1 pad 35: unconnected-(U1-ADC_VREF-Pad35) -> BB_PS
- U1 pad 36: 3V3 -> VBUS_SENSE
- U1 pad 37: PWR_EN -> unconnected-(U1-GPIO25-Pad37)
- U1 pad 38: GND -> 3V3
- U1 pad 39: VSYS -> 1V1
- U1 pad 40: unconnected-(U1-VBUS-Pad40) -> LCD_TE
- U1 pad 6: DPAD_LEFT -> 1V1
- U1 pad 7: LCD_DC -> DPAD_LEFT
- U1 pad 8: GND -> LCD_DC
Routing:
- net VBUS: track 0.00 -> 85.0 mm, vias 0 -> 3
- net RUN: track 0.00 -> 68.3 mm, vias 0 -> 2
- net SWDIO: track 0.00 -> 62.6 mm, vias 0 -> 2
- net VSYS_ADC: track 0.00 -> 62.1 mm, vias 0 -> 2
- net USB_BOOT: track 0.00 -> 53.3 mm
- net VBUS_SENSE: track 0.00 -> 48.9 mm, vias 0 -> 2
- net AUDIO_L: track 115.9 -> 75.0 mm, vias 3 -> 4
- net INR: track 6.30 -> 45.0 mm, vias 0 -> 2
- net JACK_DETSW: track 74.6 -> 39.5 mm, vias 1 -> 0
- net SWCLK: track 0.00 -> 33.9 mm, vias 0 -> 2
- net AUDIO_R: track 99.6 -> 68.2 mm
- net 3V3: track 2.60 -> 32.0 mm, vias 14 -> 29
- net OPL_N: track 52.6 -> 23.9 mm, vias 0 -> 3
- net OPR_N: track 56.8 -> 28.2 mm
- net GND: track 9.49 -> 37.5 mm, vias 49 -> 113
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- added copper zone on B.Cu, net 1V1
- added copper zone on B.Cu, net 3V3
- added copper zone on B.Cu, net GND
- added copper zone on B.Cu, net VREG_LX
