File: hardware/pikocore_gamepad/pcb/02_mcu_controles.kicad_sch (KiCad schematic)
At the start: 20 parts, among them J4 LCD_FPC, Q1 2N7002, SW1 DPAD_UP, SW10 BTN_R, SW11 BTN_START, SW12 BTN_SELECT, SW2 DPAD_DOWN, SW3 DPAD_LEFT, SW4 DPAD_RIGHT, SW5 BTN_X, SW6 BTN_Y, SW7 BTN_A, SW8 BTN_B, SW9 BTN_L, U1 RP2350-Plus-16MB

Commit message: hw: RP2350A chip-down en la placa (reemplaza el modulo RP2350-Plus)
El modulo Waveshare RP2350-Plus sale y su circuito pasa al dorso:
RP2350A QFN-60 con el nucleo de la placa minima oficial de Raspberry Pi
(MIT) copiado como bloque rigido (import_rp_minimal.py -> rp_core_ref.py,
colocado por rp_core.py), flash W25Q128, cristal 12 MHz, USB-C, cargador
ETA6096, OR de alimentacion con MBR230, buck-boost TPS63001 a 3V3,
botones BOOTSEL/RUN y pads SWD. GP0-22/GP26 sin cambios; GP23/24/29
nuevos (BB_PS, VBUS_SENSE, VSYS_ADC) tambien en config.h.

Ruteo:
- El cobre previo (nucleo, pistas manuales, vias a plano) va al DSN
  protegido; las zonas del nucleo en la cara del chip van como keepout.
- Segunda pasada de freerouting solo si deja menos conexiones abiertas.
- Senales a 0.127/0.127 con via 0.45/0.2; Power con via propia 0.6/0.3.
- Carriles de salida de la placa oficial para LCD_DC, LCD_MOSI,
  BTN_START y DPAD_UP/DOWN; pin 1 de U1 al anillo de 3V3 a mano.
- TPS63001 a 180 grados con L1/L2 a mano; GND y VBUS del USB-C a mano.

Puertas: 191 tests, ERC 0, DRC 0 errores / 0 sin conectar / 0 paridad
(9 avisos previos), G-5/G-4/G-2/placement en verde. G-0 sigue en rojo
solo por LCD_FPC_PIN_ORDER, como en main. Sin verificar: LCSC de R31
(ISET 150k), saturacion de L4, rotaciones del CPL de las piezas nuevas.

Co-Authored-By: Claude Opus 5.5 <noreply@anthropic.com>
Parts:
- removed U1: RP2350-Plus-16MB, gamesetup_fp:RP2350-Plus_Socket, symbol pikocore_gamepad:RP2350-Plus
Connections:
- no-connect marks 4 -> 1

Commit message: hw: hoja 07_midi en el esquematico
Co-Authored-By: Claude Fable 5.1 <noreply@anthropic.com>
Parts:
- removed LCD1: DM-TFT13-377-24P, gamesetup_fp:LCD_LH133T_24P, symbol pikocore_gamepad:LCD_PANEL
- added C30: 1uF, Capacitor_SMD:C_0603_1608Metric, symbol pikocore_gamepad:C
- LCD1: renamed from C30; value 1uF -> DM-TFT13-377-24P; footprint Capacitor_SMD:C_0603_1608Metric -> gamesetup_fp:LCD_LH133T_24P; symbol pikocore_gamepad:C -> pikocore_gamepad:LCD_PANEL; LCSC C15849 -> (none); now not fitted
Connections:
- net 3V3: now also C30.1; no longer LCD1.1
- net GND: now also C30.2; no longer LCD1.2
Changed lines of the file:
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@@
     (date "2026-08-28")
     (rev "A")
-    (comment 1 "pikocore_gamepad - hoja 3 de 7")
+    (comment 1 "pikocore_gamepad - hoja 3 de 8")
     (comment 2 "Todas las conexiones son por GLOBAL LABEL: valen en todas las hojas")
   )
