File: hardware/pikocore_gamepad/pcb/06_mcu_nucleo.kicad_sch (KiCad schematic)
At the start: 31 parts, among them SW13 BOOTSEL, SW14 RUN, U1 RP2350A, U6 W25Q128JVSIQ, Y1 12MHz

Commit message: hw: hoja 07_midi en el esquematico
Co-Authored-By: Claude Fable 5.1 <noreply@anthropic.com>
Connections:
- net VBUS_SENSE: now also U1.41 (GPIO27); no longer U1.36 (GPIO24)
- net MIDI_RX: now reaches U1.37 (GPIO25)
- new net MIDI_TX: U1.36 (GPIO24)
- no-connect marks 3 -> 1
Changed lines of the file:
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@@
     (date "2026-08-28")
     (rev "A")
-    (comment 1 "pikocore_gamepad - hoja 4 de 7")
+    (comment 1 "pikocore_gamepad - hoja 4 de 8")
     (comment 2 "Todas las conexiones son por GLOBAL LABEL: valen en todas las hojas")
   )
@@
     (property "Intersheetrefs" "${INTERSHEET_REFS}" (at 76.2 99.06 0) (effects (font (size 1.27 1.27)) (hide yes)))
   )
-  (global_label "VBUS_SENSE" (shape passive) (at 76.2 96.52 0)
+  (global_label "MIDI_TX" (shape passive) (at 76.2 96.52 0)
     (effects (font (size 1.27 1.27)) (justify left))
     (property "Intersheetrefs" "${INTERSHEET_REFS}" (at 76.2 96.52 0) (effects (font (size 1.27 1.27)) (hide yes)))
   )
-  (no_connect (at 76.2 93.98))
+  (global_label "MIDI_RX" (shape passive) (at 76.2 93.98 0)
+    (effects (font (size 1.27 1.27)) (justify left))
+    (property "Intersheetrefs" "${INTERSHEET_REFS}" (at 76.2 93.98 0) (effects (font (size 1.27 1.27)) (hide yes)))
+  )
   (global_label "3V3" (shape passive) (at 76.2 91.44 0)
     (effects (font (size 1.27 1.27)) (justify left))
@@
     (property "Intersheetrefs" "${INTERSHEET_REFS}" (at 76.2 86.36 0) (effects (font (size 1.27 1.27)) (hide yes)))
   )
-  (no_connect (at 76.2 83.82))
+  (global_label "VBUS_SENSE" (shape passive) (at 76.2 83.82 0)
+    (effects (font (size 1.27 1.27)) (justify left))
+    (property "Intersheetrefs" "${INTERSHEET_REFS}" (at 76.2 83.82 0) (effects (font (size 1.27 1.27)) (hide yes)))
+  )
   (no_connect (at 76.2 81.28))
   (global_label "VSYS_ADC" (shape passive) (at 76.2 78.74 0)
