File: hardware/pikocore_gamepad/pcb/07_midi.kicad_sch (KiCad schematic)
At the start: 10 parts, among them J6 MIDI IN, J7 MIDI OUT, U10 H11L1M, U9 74LVC1G17

Commit message: hw: codigos LCSC de las piezas del MIDI, verificados en lcsc.com
C22859 10R, C23140 33R, C22962 220R (UNI-ROYAL 0603 1%), C81598 1N4148W
(ST Semtech, SOD-123), C10425 SN74LVC1G17DCKR (SC-70-5), C20082
H11L1SR2M (onsemi, gull-wing SMD en carrete; el C16587 es el DIP
pasante). El paquete de fab queda con las 20 lineas sin codigo que ya
tenia main (piezas de soldadura manual).

Co-Authored-By: Claude Fable 5.1 <noreply@anthropic.com>
Parts:
- D3: LCSC (none) -> C81598
- R40: LCSC (none) -> C23140
- R41: LCSC (none) -> C22859
- R42: LCSC (none) -> C22962
- U10: value H11L1M -> H11L1SR2M; LCSC (none) -> C20082
- U9: value 74LVC1G17 -> SN74LVC1G17DCKR; LCSC (none) -> C10425
Changed lines of the file:
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@@
     (exclude_from_sim no) (in_bom yes) (on_board yes) (dnp no)
     (property "Reference" "U10" (at 53.34 26.67 0) (effects (font (size 1.27 1.27))))
-    (property "Value" "H11L1M" (at 53.34 54.61 0) (effects (font (size 1.27 1.27))))
+    (property "Value" "H11L1SR2M" (at 53.34 54.61 0) (effects (font (size 1.27 1.27))))
     (property "Footprint" "Package_DIP:SMDIP-6_W7.62mm" (at 53.34 40.64 0) (effects (font (size 1.27 1.27)) (hide yes)))
     (property "Datasheet" "https://www.onsemi.com/products/interfaces/optocouplers/h11l1m" (at 53.34 40.64 0) (effects (font (size 1.27 1.27)) (hide yes)))
     (property "Description" "Optoacoplador con salida Schmitt (onsemi H11L1M, SMDIP-6). PINOUT VERIFICADO contra el datasheet Fairchild/onsemi H11L1M Rev. 1.0.7 (septiembre 2014, figura 1, esquema): 1 anodo, 2 catodo, 3 sin conexion, 4 VO (colector abierto, hunde 16mA a 0.4V), 5 GND, 6 VCC. Copia en hardware/pikocore_gamepad/datasheets/." (at 53.34 40.64 0) (effects (font (size 1.27 1.27)) (hide yes)))
+    (property "LCSC" "C20082" (at 53.34 40.64 0) (effects (font (size 1.27 1.27)) (hide yes)))
     (pin "1")
     (pin "2")
@@
     (exclude_from_sim no) (in_bom yes) (on_board yes) (dnp no)
     (property "Reference" "U9" (at 251.46 29.21 0) (effects (font (size 1.27 1.27))))
-    (property "Value" "74LVC1G17" (at 251.46 52.07 0) (effects (font (size 1.27 1.27))))
+    (property "Value" "SN74LVC1G17DCKR" (at 251.46 52.07 0) (effects (font (size 1.27 1.27))))
     (property "Footprint" "Package_TO_SOT_SMD:SOT-353_SC-70-5" (at 251.46 40.64 0) (effects (font (size 1.27 1.27)) (hide yes)))
     (property "Datasheet" "https://www.ti.com/lit/ds/symlink/sn74lvc1g17.pdf" (at 251.46 40.64 0) (effects (font (size 1.27 1.27)) (hide yes)))
     (property "Description" "Buffer Schmitt de una compuerta SN74LVC1G17 (SC-70-5 / DCK). Toma los 5mA del lazo MIDI en vez del GPIO. PINOUT VERIFICADO contra el datasheet de TI SCES351Y (rev. octubre 2025, pagina 3, tabla Pin Functions, columna DBV/DCK/DRL/DPW): 1 NC, 2 A, 3 GND, 4 Y, 5 VCC. VCC 1.65-5.5V; IOL/IOH 16mA a 3V (el lazo MIDI pide 5)." (at 251.46 40.64 0) (effects (font (size 1.27 1.27)) (hide yes)))
+    (property "LCSC" "C10425" (at 251.46 40.64 0) (effects (font (size 1.27 1.27)) (hide yes)))
     (pin "1")
     (pin "2")
@@
     (property "Datasheet" "" (at 317.5 40.64 0) (effects (font (size 1.27 1.27)) (hide yes)))
     (property "Description" "Diodo de senal 1N4148W (SOD-123). Pin 1 = CATODO, como todos los footprints de diodo de KiCad; pin 2 = anodo. Antiparalelo al LED del opto de MIDI IN: protege contra un cable con polaridad al reves." (at 317.5 40.64 0) (effects (font (size 1.27 1.27)) (hide yes)))
+    (property "LCSC" "C81598" (at 317.5 40.64 0) (effects (font (size 1.27 1.27)) (hide yes)))
     (pin "1")
     (pin "2")
@@
     (property "Datasheet" "" (at 119.38 81.28 0) (effects (font (size 1.27 1.27)) (hide yes)))
     (property "Description" "Resistencia SMD 0603" (at 119.38 81.28 0) (effects (font (size 1.27 1.27)) (hide yes)))
+    (property "LCSC" "C23140" (at 119.38 81.28 0) (effects (font (size 1.27 1.27)) (hide yes)))
     (pin "1")
     (pin "2")
@@
     (property "Datasheet" "" (at 185.42 81.28 0) (effects (font (size 1.27 1.27)) (hide yes)))
     (property "Description" "Resistencia SMD 0603" (at 185.42 81.28 0) (effects (font (size 1.27 1.27)) (hide yes)))
+    (property "LCSC" "C22859" (at 185.42 81.28 0) (effects (font (size 1.27 1.27)) (hide yes)))
     (pin "1")
     (pin "2")
@@
     (property "Datasheet" "" (at 251.46 81.28 0) (effects (font (size 1.27 1.27)) (hide yes)))
     (property "Description" "Resistencia SMD 0603" (at 251.46 81.28 0) (effects (font (size 1.27 1.27)) (hide yes)))
+    (property "LCSC" "C22962" (at 251.46 81.28 0) (effects (font (size 1.27 1.27)) (hide yes)))
     (pin "1")
     (pin "2")
