File: hardware/pikocore_gamepad/pcb/01_alimentacion.kicad_sch (KiCad schematic)
At the start: 10 parts, among them SW15 PWR, U2 TPS61023DRLR

Commit message: hw: RP2350A chip-down en la placa (reemplaza el modulo RP2350-Plus)
El modulo Waveshare RP2350-Plus sale y su circuito pasa al dorso:
RP2350A QFN-60 con el nucleo de la placa minima oficial de Raspberry Pi
(MIT) copiado como bloque rigido (import_rp_minimal.py -> rp_core_ref.py,
colocado por rp_core.py), flash W25Q128, cristal 12 MHz, USB-C, cargador
ETA6096, OR de alimentacion con MBR230, buck-boost TPS63001 a 3V3,
botones BOOTSEL/RUN y pads SWD. GP0-22/GP26 sin cambios; GP23/24/29
nuevos (BB_PS, VBUS_SENSE, VSYS_ADC) tambien en config.h.

Ruteo:
- El cobre previo (nucleo, pistas manuales, vias a plano) va al DSN
  protegido; las zonas del nucleo en la cara del chip van como keepout.
- Segunda pasada de freerouting solo si deja menos conexiones abiertas.
- Senales a 0.127/0.127 con via 0.45/0.2; Power con via propia 0.6/0.3.
- Carriles de salida de la placa oficial para LCD_DC, LCD_MOSI,
  BTN_START y DPAD_UP/DOWN; pin 1 de U1 al anillo de 3V3 a mano.
- TPS63001 a 180 grados con L1/L2 a mano; GND y VBUS del USB-C a mano.

Puertas: 191 tests, ERC 0, DRC 0 errores / 0 sin conectar / 0 paridad
(9 avisos previos), G-5/G-4/G-2/placement en verde. G-0 sigue en rojo
solo por LCD_FPC_PIN_ORDER, como en main. Sin verificar: LCSC de R31
(ISET 150k), saturacion de L4, rotaciones del CPL de las piezas nuevas.

Co-Authored-By: Claude Opus 5.5 <noreply@anthropic.com>
Parts:
- added C48: 1uF, Capacitor_SMD:C_0603_1608Metric, symbol pikocore_gamepad:C
- added C49, C6: 22uF, Capacitor_SMD:C_0805_2012Metric, symbol pikocore_gamepad:C
- added C50, C51, C52, C53: 10uF, Capacitor_SMD:C_0603_1608Metric, symbol pikocore_gamepad:C
- added C54, C55: 100nF, Capacitor_SMD:C_0603_1608Metric, symbol pikocore_gamepad:C
- added D1, D2: MBR230LSFT1G, Diode_SMD:D_SOD-123F, symbol pikocore_gamepad:D_Schottky
- added J2: USB-C, Connector_USB:USB_C_Receptacle_HCTL_HC-TYPE-C-16P-01A, symbol pikocore_gamepad:USB_C16
- added J3: LiPo, Connector_Molex:Molex_PicoBlade_53398-0271_1x02-1MP_P1.25mm_Vertical, symbol pikocore_gamepad:Conn_Bat
- added L4, L5: 2.2uH, Inductor_SMD:L_1210_3225Metric, symbol pikocore_gamepad:L
- added R29, R30: 5.1k, Resistor_SMD:R_0603_1608Metric, symbol pikocore_gamepad:R
- added R31: 150k, Resistor_SMD:R_0603_1608Metric, symbol pikocore_gamepad:R
- added R32: 100R, Resistor_SMD:R_0603_1608Metric, symbol pikocore_gamepad:R
- added R33, R35, R38: 100k, Resistor_SMD:R_0603_1608Metric, symbol pikocore_gamepad:R
- added R34: 10k, Resistor_SMD:R_0603_1608Metric, symbol pikocore_gamepad:R
- added R36, R37, R4: 200k, Resistor_SMD:R_0603_1608Metric, symbol pikocore_gamepad:R
- U7: renamed from C6; value 22uF -> TPS63001DRCR; footprint Capacitor_SMD:C_0805_2012Metric -> Package_SON:Texas_DRC0010J_ThermalVias; symbol pikocore_gamepad:C -> pikocore_gamepad:TPS63001; LCSC C45783 -> C28060
- U8: renamed from R4; value 200k -> ETA6096D3K; footprint Resistor_SMD:R_0603_1608Metric -> gamesetup_lcsc:DFN-10_L3.0-W3.0-P0.50-BL-EP2.4-1; symbol pikocore_gamepad:R -> pikocore_gamepad:ETA6096; LCSC C25811 -> C7465538
Connections:
- net 5V: now also C6.1, R4.1; no longer U7.1, U8.1
- net BOOST_FB: now also R4.2; no longer U8.2
- net GND: now also U7.11 (EP), U7.3 (PGND), U7.9 (GND), U8.10 (AGND), U8.11 (EP), U8.3 (PGND), U8.7 (AGND), C48.2, C49.2, C50.2, C51.2, C52.2, C53.2, C54.2, C55.2, C6.2, J2.A1, J2.A12, J2.B1, J2.B12, J2.S1, J3.2 (BAT-), J3.MP, R29.2, R30.2, R31.2, R34.2, R36.2, R38.2; no longer U7.2
- net PWR_EN: now also U7.6 (EN), R33.2
- net VSYS: now also U7.5 (VIN), C51.1, D1.1 (K), D2.1 (K), R32.1, R33.1, R37.1
- new net 3V3: C52.1, C53.1, U7.1 (VOUT), U7.10 (FB)
- new net BB_L1: L5.1, U7.4 (L1)
- new net BB_L2: L5.2, U7.2 (L2)
- new net BB_PS: R34.1, U7.7 (PS)
- new net BB_VINA: C54.1, R32.2, U7.8 (VINA)
- new net CHG_ISET: R31.1, U8.8 (ISET)
- new net CHG_PMID: C49.1, U8.2 (PMID)
- new net CHG_SW: L4.1, U8.5 (SW)
- new net USB_CC1: J2.A5, R29.1
- new net USB_CC2: J2.B5, R30.1
- new net USB_DM: J2.A7, J2.B7
- new net USB_DP: J2.A6, J2.B6
- new net VBAT: C50.1, D2.2 (A), J3.1 (BAT+), L4.2, U8.6 (BATS)
- new net VBUS: C48.1, D1.2 (A), J2.A4, J2.A9, J2.B4, J2.B9, R35.1, U8.1 (VIN)
- new net VBUS_SENSE: R35.2, R36.1
- new net VSYS_ADC: C55.1, R37.2, R38.1
- no-connect marks 1 -> 5
Other:
- note added: "VSYS = la mayor entre VBUS (USB) y VBAT (LiPo), cada una por un Schottky (D1, D2). El cargador U8 toma VBUS antes del diodo. ISET 150k = 1.2A (datasheet). El 3V3 lo hace el buck-boost U7 (TPS63001, salida fija) desde VSYS: sigue en 3.3V con la LiPo descargada. PS/SYNC con pulldown (power-save); GP23 lo sube para PWM fijo. VBUS/3*2 a GP24 (sensado de USB) y VSYS/3 a GP29 (ADC3, nivel de bateria). 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"
- note removed: "El riel de 5V alimenta SOLO al op-amp U3 (hoja 4). Es a proposito: el riel analogico tiene que ser FIJO y no seguir a la bateria, porque la masa virtual del op-amp se deriva de el. El class-D U4 (hoja 5) NO cuelga de aca sino de VSYS directo, porque a todo volumen pide cientos de mA y hacerlo pasar por el boost obligaria a dimensionarlo para el pico del parlante. Divisor de realimentacion: Vout =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"
- title: Alimentacion - boost 5V y encendido -> Alimentacion - USB, carga, 3V3, boost 5V y encendido

Commit message: hw: cierra R31, L4 y rotaciones del CPL del chip-down
- R31 (ISET 150k 0603) -> C22807 (UNI-ROYAL 0603WAF1503T5E) en LCSC_PASIVOS.
  Esquematico y .net regenerados: solo cambia el campo LCSC.
- L4 (C3002559, CENKER CKST322512-2.2uH): Isat 4.0A contra un pico de
  ~1.9A (2.35A a 300kHz) a 1.2A de carga. Sin cambio.
- gen_fab: el CPL espeja el angulo de las piezas del dorso
  ((180 - rot) + correccion) y aplica CORRECCIONES_CPL por footprint,
  verificadas contra el footprint EasyEDA de cada LCSC: U6 SOIC +270,
  J2 USB-C centro corrido 1.335mm. Test en tests/test_gen_fab.py.

Sin reruteo. Puertas: 194 tests OK, ERC 0, DRC 0 errores / 0 sin
conectar / 0 paridad, G-0 rojo solo por LCD_FPC_PIN_ORDER.

Co-Authored-By: Claude Opus 5.5 <noreply@anthropic.com>
Parts:
- R31: LCSC (none) -> C22807
Changed lines of the file:
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@@
     (property "Datasheet" "" (at 251.46 327.66 0) (effects (font (size 1.27 1.27)) (hide yes)))
     (property "Description" "Resistencia SMD 0603" (at 251.46 327.66 0) (effects (font (size 1.27 1.27)) (hide yes)))
+    (property "LCSC" "C22807" (at 251.46 327.66 0) (effects (font (size 1.27 1.27)) (hide yes)))
     (pin "1")
     (pin "2")

Commit message: hw: bateria con conector JST GH (las celdas del usuario no son MX1.25)
J3 pasa de Molex PicoBlade a JST GH BM02B-GHS-TBT (1.25mm, vertical SMD,
con traba), LCSC C161690 verificado en lcsc.com. Las celdas del usuario
traen GH, que no entra en el PicoBlade aunque tenga el mismo paso.
Posicion corrida a x 4.6 por el courtyard mas ancho; ciclo de ruteo
completo, DRC 0 errores / 0 sin conectar / 0 paridad.

Co-Authored-By: Claude Sonnet 5.5 <noreply@anthropic.com>
Parts:
- J3: footprint Connector_Molex:Molex_PicoBlade_53398-0271_1x02-1MP_P1.25mm_Vertical -> Connector_JST:JST_GH_BM02B-GHS-TBT_1x02-1MP_P1.25mm_Vertical; LCSC (none) -> C161690
Changed lines of the file:
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@@
     (property "Reference" "J3" (at 53.34 95.25 0) (effects (font (size 1.27 1.27))))
     (property "Value" "LiPo" (at 53.34 113.03 0) (effects (font (size 1.27 1.27))))
-    (property "Footprint" "Connector_Molex:Molex_PicoBlade_53398-0271_1x02-1MP_P1.25mm_Vertical" (at 53.34 104.14 0) (effects (font (size 1.27 1.27)) (hide yes)))
-    (property "Datasheet" "" (at 53.34 104.14 0) (effects (font (size 1.27 1.27)) (hide yes)))
-    (property "Description" "Conector de bateria Molex PicoBlade 1.25mm 2P vertical SMD (compatible MX1.25). 1 = +, 2 = -, MP = lenguetas de anclaje. OJO: las LiPo con este conector vienen en las dos polaridades." (at 53.34 104.14 0) (effects (font (size 1.27 1.27)) (hide yes)))
+    (property "Footprint" "Connector_JST:JST_GH_BM02B-GHS-TBT_1x02-1MP_P1.25mm_Vertical" (at 53.34 104.14 0) (effects (font (size 1.27 1.27)) (hide yes)))
+    (property "Datasheet" "https://www.lcsc.com/product-detail/C161690.html" (at 53.34 104.14 0) (effects (font (size 1.27 1.27)) (hide yes)))
+    (property "Description" "Conector de bateria JST GH 1.25mm 2P vertical SMD (BM02B-GHS-TBT, con traba): es el que traen las celdas del usuario y NO entra en el PicoBlade/MX1.25 aunque tenga el mismo paso (2026-10-16). 1 = +, 2 = -, MP = lenguetas de anclaje. OJO: las LiPo vienen en las dos polaridades." (at 53.34 104.14 0) (effects (font (size 1.27 1.27)) (hide yes)))
+    (property "LCSC" "C161690" (at 53.34 104.14 0) (effects (font (size 1.27 1.27)) (hide yes)))
     (pin "1")
     (pin "2")
