File: hardware/pikocore_gamepad/pcb/04_opamp.kicad_sch (KiCad schematic)
At the start: 13 parts, among them U3 PT2308-S

Commit message: hw: paquete de fabricación con las 4 capas, paridad esquemático↔PCB en 0
gen_fab.py pedía las capas internas por su nombre de usuario (GND/PWR);
kicad-cli 9.0.1 las rechazaba con un aviso y exit 0, y el zip salía con
dos capas de cobre para una placa de cuatro. Ahora usa In1.Cu/In2.Cu y
aborta si falta cualquier gerber obligatorio. También busca kicad-cli en
Program Files, que es donde está en esta máquina.

gen_pcb.py dejaba el FPID sin librería y el Value con el nombre del
footprint: 128 avisos footprint_symbol_mismatch en el DRC con
--schematic-parity. identidad_desde_netlist() los pone desde netlist.py
y finish_pcb.py lo repite al final del ciclo, así la placa ya ruteada
quedó corregida sin re-rutear. C23/C24 (soldadura manual) van DNP
también en el esquemático.

Estado tras la corrida completa de pcb-verify: 201 tests, G-0/G-5/G-4/
G-2/placement OK, ERC 0 errores, DRC 0 errores / 0 nets sin rutear /
0 paridad. README de hardware y checklist JLCPCB actualizados.

Co-Authored-By: Claude Fable 5.1 <noreply@anthropic.com>
Parts:
- C23, C24: MANUAL True -> (none); now not fitted
Changed lines of the file:
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@@
     (at 53.34 81.28 0)
     (unit 1)
-    (exclude_from_sim no) (in_bom yes) (on_board yes) (dnp no)
+    (exclude_from_sim no) (in_bom yes) (on_board yes) (dnp yes)
     (property "Reference" "C23" (at 53.34 69.85 0) (effects (font (size 1.27 1.27))))
     (property "Value" "470uF" (at 53.34 92.71 0) (effects (font (size 1.27 1.27))))
@@
     (property "Datasheet" "" (at 53.34 81.28 0) (effects (font (size 1.27 1.27)) (hide yes)))
     (property "Description" "Capacitor electrolitico. POLARIZADO: montado al reves revienta, por eso tiene simbolo propio y no se mezcla con los ceramicos." (at 53.34 81.28 0) (effects (font (size 1.27 1.27)) (hide yes)))
-    (property "MANUAL" "True" (at 53.34 81.28 0) (effects (font (size 1.27 1.27)) (hide yes)))
     (pin "1")
     (pin "2")
@@
     (at 119.38 81.28 0)
     (unit 1)
-    (exclude_from_sim no) (in_bom yes) (on_board yes) (dnp no)
+    (exclude_from_sim no) (in_bom yes) (on_board yes) (dnp yes)
     (property "Reference" "C24" (at 119.38 69.85 0) (effects (font (size 1.27 1.27))))
     (property "Value" "470uF" (at 119.38 92.71 0) (effects (font (size 1.27 1.27))))
@@
     (property "Datasheet" "" (at 119.38 81.28 0) (effects (font (size 1.27 1.27)) (hide yes)))
     (property "Description" "Capacitor electrolitico. POLARIZADO: montado al reves revienta, por eso tiene simbolo propio y no se mezcla con los ceramicos." (at 119.38 81.28 0) (effects (font (size 1.27 1.27)) (hide yes)))
-    (property "MANUAL" "True" (at 119.38 81.28 0) (effects (font (size 1.27 1.27)) (hide yes)))
     (pin "1")
     (pin "2")
